Commit message: SLAM package adpatable for any robot

File: TurtleBot/turtlebot3_gazebo/urdf/turtlebot3_burger.urdf (robot description, URDF)
Before this commit: robot turtlebot3_burger, 7 links, 6 joints
Links:
- removed link tb3/base_footprint
- removed link tb3/base_link
- removed link tb3/base_scan
- removed link tb3/caster_back_link
- removed link tb3/imu_link
- removed link tb3/wheel_left_link
- removed link tb3/wheel_right_link
- added link tb3_base_footprint
- added link tb3_base_link, mass 8.2573504e-01; collision box size=0.140 0.140 0.143; visual mesh filename=package://turtlebot3_gazebo/models/turtlebot3_common/meshes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 scale=0.001 0.001 0.001
- added link tb3_base_scan, mass 0.114; collision cylinder length=0.0315 radius=0.055; visual mesh filename=package://turtlebot3_gazebo/models/turtlebot3_common/meshes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 scale=0.001 0.001 0.001
- added link tb3_caster_back_link, mass 0.005; collision box size=0.030 0.009 0.020
- added link tb3_imu_link
- added link tb3_wheel_left_link, mass 2.8498940e-02; collision cylinder length=0.018 radius=0.033; visual mesh filename=package://turtlebot3_gazebo/models/turtlebot3_common/meshes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 scale=0.001 0.001 0.001
- added link tb3_wheel_right_link, mass 2.8498940e-02; collision cylinder length=0.018 radius=0.033; visual mesh filename=package://turtlebot3_gazebo/models/turtlebot3_common/meshes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 scale=0.001 0.001 0.001
Joints:
- joint base_joint: child tb3/base_link -> tb3_base_link; parent tb3/base_footprint -> tb3_base_footprint
- joint caster_back_joint: child tb3/caster_back_link -> tb3_caster_back_link; parent tb3/base_link -> tb3_base_link
- joint imu_joint: child tb3/imu_link -> tb3_imu_link; parent tb3/base_link -> tb3_base_link
- joint scan_joint: child tb3/base_scan -> tb3_base_scan; parent tb3/base_link -> tb3_base_link
- joint wheel_left_joint: child tb3/wheel_left_link -> tb3_wheel_left_link; parent tb3/base_link -> tb3_base_link
- joint wheel_right_joint: child tb3/wheel_right_link -> tb3_wheel_right_link; parent tb3/base_link -> tb3_base_link

File: TurtleBot/turtlebot3_gazebo/urdf/turtlebot3_burger2.urdf (robot description, URDF)
Before this commit: robot turtlebot3_burger, 7 links, 6 joints
Links:
- removed link tb3_2/base_footprint
- removed link tb3_2/base_link
- removed link tb3_2/base_scan
- removed link tb3_2/caster_back_link
- removed link tb3_2/imu_link
- removed link tb3_2/wheel_left_link
- removed link tb3_2/wheel_right_link
- added link tb3_2_base_footprint
- added link tb3_2_base_link, mass 8.2573504e-01; collision box size=0.140 0.140 0.143; visual mesh filename=package://turtlebot3_gazebo/models/turtlebot3_common/meshes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 scale=0.001 0.001 0.001
- added link tb3_2_base_scan, mass 0.114; collision cylinder length=0.0315 radius=0.055; visual mesh filename=package://turtlebot3_gazebo/models/turtlebot3_common/meshes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 scale=0.001 0.001 0.001
- added link tb3_2_caster_back_link, mass 0.005; collision box size=0.030 0.009 0.020
- added link tb3_2_imu_link
- added link tb3_2_wheel_left_link, mass 2.8498940e-02; collision cylinder length=0.018 radius=0.033; visual mesh filename=package://turtlebot3_gazebo/models/turtlebot3_common/meshes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 scale=0.001 0.001 0.001
- added link tb3_2_wheel_right_link, mass 2.8498940e-02; collision cylinder length=0.018 radius=0.033; visual mesh filename=package://turtlebot3_gazebo/models/turtlebot3_common/meshes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 scale=0.001 0.001 0.001
Joints:
- joint base_joint: child tb3_2/base_link -> tb3_2_base_link; parent tb3_2/base_footprint -> tb3_2_base_footprint
- joint caster_back_joint: child tb3_2/caster_back_link -> tb3_2_caster_back_link; parent tb3_2/base_link -> tb3_2_base_link
- joint imu_joint: child tb3_2/imu_link -> tb3_2_imu_link; parent tb3_2/base_link -> tb3_2_base_link
- joint scan_joint: child tb3_2/base_scan -> tb3_2_base_scan; parent tb3_2/base_link -> tb3_2_base_link
- joint wheel_left_joint: child tb3_2/wheel_left_link -> tb3_2_wheel_left_link; parent tb3_2/base_link -> tb3_2_base_link
- joint wheel_right_joint: child tb3_2/wheel_right_link -> tb3_2_wheel_right_link; parent tb3_2/base_link -> tb3_2_base_link

Commit message: frame_prefix added, 3 robots localization

File: TurtleBot/turtlebot3_gazebo/urdf/turtlebot3_burger.urdf (robot description, URDF)
Before this commit: robot turtlebot3_burger, 7 links, 6 joints
Links:
- removed link tb3_base_footprint
- removed link tb3_base_link
- removed link tb3_base_scan
- removed link tb3_caster_back_link
- removed link tb3_imu_link
- removed link tb3_wheel_left_link
- removed link tb3_wheel_right_link
- added link base_footprint
- added link base_link, mass 8.2573504e-01; collision box size=0.140 0.140 0.143; visual mesh filename=package://turtlebot3_gazebo/models/turtlebot3_common/meshes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 scale=0.001 0.001 0.001
- added link base_scan, mass 0.114; collision cylinder length=0.0315 radius=0.055; visual mesh filename=package://turtlebot3_gazebo/models/turtlebot3_common/meshes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 scale=0.001 0.001 0.001
- added link caster_back_link, mass 0.005; collision box size=0.030 0.009 0.020
- added link imu_link
- added link wheel_left_link, mass 2.8498940e-02; collision cylinder length=0.018 radius=0.033; visual mesh filename=package://turtlebot3_gazebo/models/turtlebot3_common/meshes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 scale=0.001 0.001 0.001
- added link wheel_right_link, mass 2.8498940e-02; collision cylinder length=0.018 radius=0.033; visual mesh filename=package://turtlebot3_gazebo/models/turtlebot3_common/meshes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 scale=0.001 0.001 0.001
Joints:
- joint base_joint: child tb3_base_link -> base_link; parent tb3_base_footprint -> base_footprint
- joint caster_back_joint: child tb3_caster_back_link -> caster_back_link; parent tb3_base_link -> base_link
- joint imu_joint: child tb3_imu_link -> imu_link; parent tb3_base_link -> base_link
- joint scan_joint: child tb3_base_scan -> base_scan; parent tb3_base_link -> base_link
- joint wheel_left_joint: child tb3_wheel_left_link -> wheel_left_link; parent tb3_base_link -> base_link
- joint wheel_right_joint: child tb3_wheel_right_link -> wheel_right_link; parent tb3_base_link -> base_link
