Commit message: Gazebo use of namespace for cameras/plugin

File: realsense-ros/realsense2_description/urdf/cam_l515.urdf.xacro (robot description, xacro)
@@ -5,5 +5,10 @@
 -->
 <robot name="cam_l515" xmlns:xacro="http://ros.org/wiki/xacro">
-    <link name="base_link"/>
+    <link name="world" />
+    <link name="origin_frame"/>
+    <joint name="world_to_origin_frame" type="fixed">
+        <parent link="world"/>
+        <child link="origin_frame"/>
+    </joint>
     <!-- Import macro for realsense-RS200 camera-->
     <xacro:arg name="use_nominal_extrinsics" default="true"/>
@@ -15,5 +20,5 @@
     <xacro:include filename="$(find realsense2_description)/urdf/_l515.urdf.xacro"/>
     <!-- Create camera instance -->
-    <xacro:sensor_l515 parent="base_link" use_nominal_extrinsics="$(arg use_nominal_extrinsics)" add_plug="$(arg add_plug)" use_mesh="$(arg use_mesh)" name="$(arg name)" topics_ns="$(arg topics_ns)" publish_pointcloud="$(arg publish_pointcloud)">
+    <xacro:sensor_l515 parent="world" use_nominal_extrinsics="$(arg use_nominal_extrinsics)" add_plug="$(arg add_plug)" use_mesh="$(arg use_mesh)" name="$(arg name)" topics_ns="$(arg topics_ns)" publish_pointcloud="$(arg publish_pointcloud)">
         <origin xyz="0 0 1.0" rpy="0 0 0" />
     </xacro:sensor_l515>

Commit message: [In develop] Spawn arucos in world

File: realsense-ros/realsense2_description/urdf/cam_l515.urdf.xacro (robot description, xacro)
@@ -21,5 +21,5 @@
     <!-- Create camera instance -->
     <xacro:sensor_l515 parent="world" use_nominal_extrinsics="$(arg use_nominal_extrinsics)" add_plug="$(arg add_plug)" use_mesh="$(arg use_mesh)" name="$(arg name)" topics_ns="$(arg topics_ns)" publish_pointcloud="$(arg publish_pointcloud)">
-        <origin xyz="0 0 1.0" rpy="0 0 0" />
+        <origin xyz="0 0 1.0" rpy="1.54 0 0" />
     </xacro:sensor_l515>
 </robot>

Commit message: [In develop] Launch for multi-cam

File: realsense-ros/realsense2_description/urdf/cam_l515.urdf.xacro (robot description, xacro)
@@ -20,6 +20,6 @@
     <xacro:include filename="$(find realsense2_description)/urdf/_l515.urdf.xacro"/>
     <!-- Create camera instance -->
-    <xacro:sensor_l515 parent="world" use_nominal_extrinsics="$(arg use_nominal_extrinsics)" add_plug="$(arg add_plug)" use_mesh="$(arg use_mesh)" name="$(arg name)" topics_ns="$(arg topics_ns)" publish_pointcloud="$(arg publish_pointcloud)">
-        <origin xyz="0 0 1.0" rpy="1.54 0 0" />
+    <xacro:sensor_l515 parent="origin_frame" use_nominal_extrinsics="$(arg use_nominal_extrinsics)" add_plug="$(arg add_plug)" use_mesh="$(arg use_mesh)" name="$(arg name)" topics_ns="$(arg topics_ns)" publish_pointcloud="$(arg publish_pointcloud)">
+        <origin xyz="-0.05 0 1.0" rpy="0 1.54 0" />
     </xacro:sensor_l515>
 </robot>

Commit message: [OK] Launch for multi camera with aruco detection

File: realsense-ros/realsense2_description/urdf/cam_l515.urdf.xacro (robot description, xacro)
@@ -16,10 +16,13 @@
     <xacro:arg name="use_mesh" default="true" />
     <xacro:arg name="name" default="camera" />
-    <xacro:arg name="topics_ns" default="camera" />
+    <xacro:arg name="namespace" default="camera" />
     <xacro:arg name="publish_pointcloud" default="true" />
+    <xacro:arg name="x_pos" default="0.0" />
+    <xacro:arg name="y_pos" default="0.0" />
+    <xacro:arg name="z_pos" default="1.0" />
     <xacro:include filename="$(find realsense2_description)/urdf/_l515.urdf.xacro"/>
     <!-- Create camera instance -->
-    <xacro:sensor_l515 parent="origin_frame" use_nominal_extrinsics="$(arg use_nominal_extrinsics)" add_plug="$(arg add_plug)" use_mesh="$(arg use_mesh)" name="$(arg name)" topics_ns="$(arg topics_ns)" publish_pointcloud="$(arg publish_pointcloud)">
-        <origin xyz="-0.05 0 1.0" rpy="0 1.54 0" />
+    <xacro:sensor_l515 parent="origin_frame" use_nominal_extrinsics="$(arg use_nominal_extrinsics)" add_plug="$(arg add_plug)" use_mesh="$(arg use_mesh)" name="$(arg name)" topics_ns="$(arg namespace)" publish_pointcloud="$(arg publish_pointcloud)">
+        <origin xyz="$(arg x_pos) $(arg y_pos) $(arg z_pos)" rpy="0 1.54 0" />
     </xacro:sensor_l515>
 </robot>

Commit message: New reference "World"

File: realsense-ros/realsense2_description/urdf/cam_l515.urdf.xacro (robot description, xacro)
@@ -6,8 +6,9 @@
 <robot name="cam_l515" xmlns:xacro="http://ros.org/wiki/xacro">
     <link name="world" />
-    <link name="origin_frame"/>
-    <joint name="world_to_origin_frame" type="fixed">
+    <link name="$(arg name)_camera_link" />
+    <joint name="world_to_camera" type="fixed">
         <parent link="world"/>
-        <child link="origin_frame"/>
+        <child link="$(arg name)_camera_link"/>
+        <origin xyz="$(arg x_pos) $(arg y_pos) $(arg z_pos)" rpy="0 1.54 0" />
     </joint>
     <!-- Import macro for realsense-RS200 camera-->
@@ -23,6 +24,6 @@
     <xacro:include filename="$(find realsense2_description)/urdf/_l515.urdf.xacro"/>
     <!-- Create camera instance -->
-    <xacro:sensor_l515 parent="origin_frame" use_nominal_extrinsics="$(arg use_nominal_extrinsics)" add_plug="$(arg add_plug)" use_mesh="$(arg use_mesh)" name="$(arg name)" topics_ns="$(arg namespace)" publish_pointcloud="$(arg publish_pointcloud)">
-        <origin xyz="$(arg x_pos) $(arg y_pos) $(arg z_pos)" rpy="0 1.54 0" />
+    <xacro:sensor_l515 parent="$(arg name)_camera_link" use_nominal_extrinsics="$(arg use_nominal_extrinsics)" add_plug="$(arg add_plug)" use_mesh="$(arg use_mesh)" name="$(arg name)" topics_ns="$(arg namespace)" publish_pointcloud="$(arg publish_pointcloud)">
+        <origin xyz="0 0 0" rpy="0 0 0" />
     </xacro:sensor_l515>
 </robot>
