Commit message: Rviz use uf namespace for cameras

File: realsense-ros/realsense2_description/urdf/_l515.gazebo.xacro (robot description, xacro)
@@ -95,10 +95,10 @@
         <colorUpdateRate>30.0</colorUpdateRate>
         <infraredUpdateRate>30.0</infraredUpdateRate>
-        <depthTopicName>/camera/depth/image_rect_raw</depthTopicName>
-        <depthCameraInfoTopicName>/camera/depth/camera_info</depthCameraInfoTopicName>
-        <colorTopicName>/camera/color/image_raw</colorTopicName>
-        <colorCameraInfoTopicName>/camera/color/camera_info</colorCameraInfoTopicName>
-        <infraredTopicName>/camera/infra/image_raw</infraredTopicName>
-        <infraredCameraInfoTopicName>/camera/infra/camera_info</infraredCameraInfoTopicName>
+        <depthTopicName>/${topics_ns}/depth/image_rect_raw</depthTopicName>
+        <depthCameraInfoTopicName>/${topics_ns}/depth/camera_info</depthCameraInfoTopicName>
+        <colorTopicName>/${topics_ns}/color/image_raw</colorTopicName>
+        <colorCameraInfoTopicName>/${topics_ns}/color/camera_info</colorCameraInfoTopicName>
+        <infraredTopicName>/${topics_ns}/infra/image_raw</infraredTopicName>
+        <infraredCameraInfoTopicName>/${topics_ns}/infra/camera_info</infraredCameraInfoTopicName>
         <colorOpticalframeName>${color_optical_frame}</colorOpticalframeName>
         <depthOpticalframeName>${depth_optical_frame}</depthOpticalframeName>
@@ -107,5 +107,5 @@
         <rangeMaxDepth>10.0</rangeMaxDepth>
         <pointCloud>${publish_pointcloud}</pointCloud>
-        <pointCloudTopicName>/camera/depth/color/points</pointCloudTopicName>
+        <pointCloudTopicName>/${topics_ns}/depth/color/points</pointCloudTopicName>
         <pointCloudCutoff>0.25</pointCloudCutoff>
         <pointCloudCutoffMax>9.0</pointCloudCutoffMax>

File: realsense-ros/realsense2_description/urdf/cam_l515.urdf.xacro (robot description, xacro)
@@ -5,9 +5,15 @@
 -->
 <robot name="cam_l515" xmlns:xacro="http://ros.org/wiki/xacro">
-    <link name="world"/>
+    <link name="base_link"/>
     <!-- Import macro for realsense-RS200 camera-->
+    <xacro:arg name="use_nominal_extrinsics" default="true"/>
+    <xacro:arg name="add_plug" default="true" />
+    <xacro:arg name="use_mesh" default="true" />
+    <xacro:arg name="name" default="camera" />
+    <xacro:arg name="topics_ns" default="camera" />
+    <xacro:arg name="publish_pointcloud" default="true" />
     <xacro:include filename="$(find realsense2_description)/urdf/_l515.urdf.xacro"/>
     <!-- Create camera instance -->
-    <xacro:sensor_l515 parent="world">
+    <xacro:sensor_l515 parent="base_link" use_nominal_extrinsics="$(arg use_nominal_extrinsics)" add_plug="$(arg add_plug)" use_mesh="$(arg use_mesh)" name="$(arg name)" topics_ns="$(arg topics_ns)" publish_pointcloud="$(arg publish_pointcloud)">
         <origin xyz="0 0 1.0" rpy="0 0 0" />
     </xacro:sensor_l515>

Commit message: New reference "map" for cameras and markers

File: realsense-ros/realsense2_description/urdf/_l515.gazebo.xacro (robot description, xacro)
@@ -13,5 +13,5 @@
       <enable_wind>0</enable_wind>
       <kinematic>0</kinematic>
-      <gravity>1</gravity>
+      <gravity>0</gravity>
       <!--<mu>1</mu>-->
       <mu2>1</mu2>

File: realsense-ros/realsense2_description/urdf/cam_l515.urdf.xacro (robot description, xacro)
@@ -5,8 +5,8 @@
 -->
 <robot name="cam_l515" xmlns:xacro="http://ros.org/wiki/xacro">
-    <link name="world" />
-    <link name="$(arg name)_camera_link" />
-    <joint name="world_to_camera" type="fixed">
-        <parent link="world"/>
+    <link name="map" />
+    <link name="$(arg name)_camera_link"/>
+    <joint name="map_to_camera" type="fixed">
+        <parent link="map"/>
         <child link="$(arg name)_camera_link"/>
         <origin xyz="$(arg x_pos) $(arg y_pos) $(arg z_pos)" rpy="0 1.54 0" />
