Commit message: [OK]Initial pose publisher for robots and added aruco marker on r1

File: Create3/create3_sim/irobot_create_common/irobot_create_description/urdf/create3.urdf.xacro (robot description, xacro)
@@ -144,4 +144,16 @@
       <xacro:inertial_cylinder mass="0.1" length="0.04" radius="0.05">
       </xacro:inertial_cylinder>
+  </link>
+  <joint name="aruco_joint" type="fixed">
+        <parent link="laser_frame"/>
+        <child link="aruco_frame"/>
+        <origin xyz="0 0 0.03" rpy="0 0 0"/>
+  </joint>
+  <link name="aruco_frame">
+      <visual>
+          <geometry>
+              <mesh filename="package://irobot_create_description/meshes/DICT_4X4_50_id15.dae"/>
+          </geometry>
+      </visual>
   </link>
   <!-- Mouse -->

Commit message: [In develop] Files for link marker in create3

File: Create3/create3_sim/irobot_create_common/irobot_create_description/urdf/create3.urdf.xacro (robot description, xacro)
@@ -148,10 +148,10 @@
         <parent link="laser_frame"/>
         <child link="aruco_frame"/>
-        <origin xyz="0 0 0.03" rpy="0 0 0"/>
+        <origin xyz="0 0 0.03" rpy="0 1.57079632679 0"/>
   </joint>
   <link name="aruco_frame">
       <visual>
           <geometry>
-              <mesh filename="package://irobot_create_description/meshes/DICT_4X4_50_id15.dae"/>
+            <mesh filename="model://marker10/meshes/Marker10.dae" scale="0.2 0.2 0.2"/>
           </geometry>
       </visual>

Commit message: New robot description with markers [(ToDo) Change the pck models]

File: Create3/create3_sim/irobot_create_common/irobot_create_description/urdf/create3.urdf.xacro (robot description, xacro)
@@ -146,12 +146,12 @@
   </link>
   <joint name="aruco_joint" type="fixed">
-        <parent link="laser_frame"/>
+        <parent link="base_link"/>
         <child link="aruco_frame"/>
-        <origin xyz="0 0 0.03" rpy="0 1.57079632679 0"/>
+        <origin xyz="-0.05 0.05 0.10" rpy="0 1.57079632679 -1.57079632679"/>
   </joint>
   <link name="aruco_frame">
       <visual>
           <geometry>
-            <mesh filename="model://marker10/meshes/Marker10.dae" scale="0.2 0.2 0.2"/>
+            <mesh filename="package://irobot_create_description/meshes/Marker10.dae" scale="0.2 0.2 0.2"/>
           </geometry>
       </visual>

Commit message: General robot description for aruco marker

File: Create3/create3_sim/irobot_create_common/irobot_create_description/urdf/create3.urdf.xacro (robot description, xacro)
@@ -15,4 +15,6 @@
   <!-- Namespace -->
   <xacro:arg name="namespace"                    default=""/>
+  <!-- ID marker -->
+  <xacro:arg name="id"                           default="10"/>
   <!-- Mechanical properties -->
   <xacro:property name="body_z_offset"           value="${-2.5*cm2m}" />
@@ -153,5 +155,5 @@
       <visual>
           <geometry>
-            <mesh filename="package://irobot_create_description/meshes/Marker10.dae" scale="0.2 0.2 0.2"/>
+            <mesh filename="package://irobot_create_description/meshes/Marker$(arg id).dae" scale="0.2 0.2 0.2"/>
           </geometry>
       </visual>

Commit message: Namespace for Odom fixed

File: Create3/create3_sim/irobot_create_common/irobot_create_description/urdf/create3.urdf.xacro (robot description, xacro)
@@ -108,7 +108,7 @@
         <parameters>$(find irobot_create_control)/config/control.yaml</parameters>
         <ros>
+          <namespace>$(arg namespace)</namespace>
           <remapping>~/odom:=odom</remapping>
           <remapping>/diagnostics:=diagnostics</remapping>
-          <namespace>$(arg namespace)</namespace>
         </ros>
       </plugin>
@@ -120,7 +120,7 @@
         <parameters>$(find irobot_create_control)/config/control.yaml</parameters>
         <ros>
+          <namespace>$(arg namespace)</namespace>
           <remapping>~/odom:=odom</remapping>
           <remapping>/diagnostics:=diagnostics</remapping>
-          <namespace>$(arg namespace)</namespace>
         </ros>
       </plugin>

File: Create3/create3_sim/irobot_create_common/irobot_create_description/urdf/sensors/cliff_sensor.urdf.xacro (robot description, xacro)
@@ -12,4 +12,5 @@
   <xacro:property name="sensor_name"         value="cliff_${name}"/>
   <xacro:property name="detection_threshold" value="${8*cm2m}"/>
+  <xacro:property name="ns"                  value="${namespace}"/>
   <joint name="${sensor_name}_joint" type="fixed">
     <xacro:insert_block name="origin"/>
@@ -27,5 +28,5 @@
       <plugin name="${sensor_name}" filename="libgazebo_ros_create_cliff_sensor.so">
         <ros>
-          <namespace>${namespace}</namespace>
+          <namespace>${ns}</namespace>
           <remapping>~/out:=_internal/${sensor_name}/event</remapping>
         </ros>

Commit message: New position for laser and aruco (with reference to imu)

File: Create3/create3_sim/irobot_create_common/irobot_create_description/urdf/create3.urdf.xacro (robot description, xacro)
@@ -45,4 +45,8 @@
   <xacro:property name="wheel_drop_z"            value="${wheel_height + wheel_drop_offset_z}"/>
   <xacro:property name="base_link_z_offset"     value="${6.42*cm2m}"/>
+  <!-- this color take effect only on rviz -->
+  <material name="red">
+    <color rgba="1.0 0.0 0.0 1.0"/> <!-- rviz green color -->
+  </material>
   <!-- Docking properties -->
   <xacro:property name="robot_model_name" value="create3"/>
@@ -130,10 +134,10 @@
         <parent link="base_link"/>
         <child link="laser_frame"/>
-        <origin xyz="0.1 0 0.175" rpy="0 0 0"/>
+        <origin xyz="-0.10 0 0.185" rpy="0 0 0"/>
   </joint>
   <link name="laser_frame">
       <visual>
           <geometry>
-              <cylinder radius="0.05" length="0.04"/>
+              <cylinder radius="0.03" length="0.03"/>
           </geometry>
           <material name="red"/>
@@ -141,14 +145,14 @@
       <collision>
           <geometry>
-              <cylinder radius="0.05" length="0.04"/>
+              <cylinder radius="0.03" length="0.03"/>
           </geometry>
       </collision>
-      <xacro:inertial_cylinder mass="0.1" length="0.04" radius="0.05">
+      <xacro:inertial_cylinder mass="0.1" length="0.03" radius="0.03">
       </xacro:inertial_cylinder>
   </link>
   <joint name="aruco_joint" type="fixed">
-        <parent link="base_link"/>
+        <parent link="imu_link"/>
         <child link="aruco_frame"/>
-        <origin xyz="-0.05 0.05 0.10" rpy="0 1.57079632679 -1.57079632679"/>
+        <origin xyz="0.0 0.05 0.01" rpy="0 1.57079632679 -1.57079632679"/>
   </joint>
   <link name="aruco_frame">
