Commit message: New Aruco models with white border

File: mrs_agents/Create3/create3_sim/irobot_create_common/irobot_create_description/urdf/create3.urdf.xacro (robot description, xacro)
@@ -154,10 +154,10 @@
         <parent link="imu_link"/>
         <child link="aruco_frame"/>
-        <origin xyz="0.0 0.05 0.01" rpy="0 1.57079632679 -1.57079632679"/>
+        <origin xyz="0.0 0.08 0.01" rpy="0 1.57079632679 -1.57079632679"/>
   </joint>
   <link name="aruco_frame">
       <visual>
           <geometry>
-            <mesh filename="package://irobot_create_description/meshes/Marker$(arg id).dae" scale="0.2 0.2 0.2"/>
+            <mesh filename="package://irobot_create_description/meshes/Marker$(arg id).dae" scale="0.3225806451612903 0.3225806451612903 0.3225806451612903"/>
           </geometry>
       </visual>
